Commit message: Phase 3 complete: Gazebo simulation with sensors and diff drive
Adds robot_simulation package (warehouse world, spawn launch, diff_drive
config), wires up Gazebo sensor plugins for LiDAR/IMU/RGB/depth camera,
fixes the diff-drive controller config loading, and adds a front caster
with corrected ground-contact height to stop the chassis tipping forward.

File: src/robot_description/urdf/visionnav_robot.urdf (robot description, URDF)
Before this commit: robot visionnav_robot, 7 links, 6 joints
Links:
- removed link caster_link
- added link caster_front_link, mass 0.1; collision sphere radius=0.05; visual sphere radius=0.05
- added link caster_rear_link, mass 0.1; collision sphere radius=0.05; visual sphere radius=0.05
- link depth_camera_link: geometry 
- link left_wheel_link: mass None -> 0.2; geometry collision cylinder length=0.04 radius=0.07; visual cylinder length=0.04 radius=0.07
- link lidar_link: geometry 
- link rgb_camera_link: geometry 
- link right_wheel_link: mass None -> 0.2; geometry collision cylinder length=0.04 radius=0.07; visual cylinder length=0.04 radius=0.07
Joints:
- removed joint caster_joint
- added joint caster_front_joint: type fixed, parent base_link, child caster_front_link, origin xyz=0.25 0 -0.12
- added joint caster_rear_joint: type fixed, parent base_link, child caster_rear_link, origin xyz=-0.25 0 -0.12
- joint left_wheel_joint: origin xyz=0 0.2 -0.1 rpy=1.5708 0 0 -> xyz=0 0.22 -0.1 rpy=0 0 0
- joint right_wheel_joint: origin xyz=0 -0.2 -0.1 rpy=1.5708 0 0 -> xyz=0 -0.22 -0.1 rpy=0 0 0
